Commit message: checking who's committed

File: walker_sim/robots/simple_walker.urdf (robot description, URDF)
Before this commit: robot bipedalWalker, 0 links, 0 joints
Links:
- added link waist, mass 0.36416

Commit message: initialize node

File: walker_sim/robots/simple_walker.urdf (robot description, URDF)
Before this commit: robot bipedalWalker, 1 links, 0 joints
Links:
- added link None

Commit message: added gazebo visual

File: walker_sim/robots/simple_walker.urdf (robot description, URDF)
Before this commit: robot bipedalWalker, 2 links, 0 joints
Links:
- removed link None
- link waist: geometry collision mesh filename=package://walker_sim/meshes/waist_L.STL; visual mesh filename=package://walker_sim/meshes/waist_L.STL

Commit message: full robot model

File: walker_sim/robots/simple_walker.urdf (robot description, URDF)
Before this commit: robot bipedal_walker, 1 links, 0 joints
Links:
- added link boom, mass 0.18809; collision mesh filename=package://walker_sim/meshes/boom_horizontal.STL
- added link footL, mass 0.0098175; collision mesh filename=package://walker_sim/meshes/contact_sensor.STL; visual mesh filename=package://walker_sim/meshes/contact_sensor.STL
- added link footR, mass 0.0098175; collision mesh filename=package://walker_sim/meshes/contact_sensor.STL; visual mesh filename=package://walker_sim/meshes/contact_sensor.STL
- added link inner_ring, mass 0.41592; collision mesh filename=package://walker_sim/meshes/inner_ring.STL
- added link outer_ring, mass 0.49244; collision mesh filename=package://walker_sim/meshes/outter_ring.STL
- added link shankL, mass 0.069508; collision mesh filename=package://walker_sim/meshes/shank.STL; visual mesh filename=package://walker_sim/meshes/shank.STL
- added link shankR, mass 0.069508; collision mesh filename=package://walker_sim/meshes/shank.STL; visual mesh filename=package://walker_sim/meshes/shank.STL
- added link thighL, mass 0.045155; collision mesh filename=package://walker_sim/meshes/31mar/thigh.STL; visual mesh filename=package://walker_sim/meshes/thigh.STL
- added link thighR, mass 0.045155; collision mesh filename=package://walker_sim/meshes/thigh.STL; visual mesh filename=package://walker_sim/meshes/thigh.STL
- added link world
Joints:
- added joint boom_waist: type prismatic, parent boom, child waist, origin xyz=0.725 0 0 rpy=0 0 0, axis 0 0 1, limit lower=-0.5 upper=0.5 effort=30 velocity=7.0
- added joint grounding: type fixed, parent world, child outer_ring, origin xyz=0 0 0 rpy=0 0 0
- added joint inner_ring_boom: type fixed, parent inner_ring, child boom, origin xyz=0 0 0.080 rpy=0 0 0, axis 0 -1 0
- added joint outer_ring_inner_ring: type prismatic, parent outer_ring, child inner_ring, origin xyz=0 0 0.330 rpy=0 0 0, axis 0 -1 0, limit lower=0.0 upper=10.0 effort=30 velocity=7.0
- added joint shankL_footL: type fixed, parent shankL, child footL, origin xyz=0 0 -0.175 rpy=0 0 0
- added joint shankR_footR: type fixed, parent shankR, child footR, origin xyz=0 0 -0.175 rpy=0 0 0
- added joint thighL_shankL: type revolute, parent thighL, child shankL, origin xyz=0 0 -0.190 rpy=0 0 0, axis 1 0 0, limit lower=-0.00118981 upper=1.4 effort=30 velocity=7.0
- added joint thighR_shankR: type revolute, parent thighR, child shankR, origin xyz=0 0 -0.190 rpy=0 0 0, axis 1 0 0, limit lower=-0.00118981 upper=1.4 effort=30 velocity=7.0
- added joint waist_thighL: type revolute, parent waist, child thighL, origin xyz=0.0775 0 0 rpy=0 0 0, axis 1 0 0, limit lower=-0.8 upper=0.8 effort=30 velocity=7.0
- added joint waist_thighR: type revolute, parent waist, child thighR, origin xyz=-0.0775 0 0 rpy=0 0 0, axis 1 0 0, limit lower=-0.8 upper=0.8 effort=30 velocity=7.0
